Commit message: Add cylinder visualization. Add Visuals to URDF files

File: data/cheetah_link0_1.urdf (robot description, URDF)
Before this commit: robot , 17 links, 16 joints
Links:
- link bfoot: geometry collision capsule length=0.18800 radius=0.04600; visual capsule length=0.18800 radius=0.04600
- link bshin: geometry collision capsule length=0.30000 radius=0.04600; visual capsule length=0.30000 radius=0.04600
- link bthigh: geometry collision capsule length=0.29000 radius=0.04600; visual capsule length=0.29000 radius=0.04600
- link ffoot: geometry collision capsule length=0.14000 radius=0.04600; visual capsule length=0.14000 radius=0.04600
- link fshin: geometry collision capsule length=0.21200 radius=0.04600; visual capsule length=0.21200 radius=0.04600
- link fthigh: geometry collision capsule length=0.26600 radius=0.04600; visual capsule length=0.26600 radius=0.04600
- link torso: geometry collision capsule length=0.30000 radius=0.04600; collision capsule length=1.00000 radius=0.04600

File: data/hopper_link0_1.urdf (robot description, URDF)
Before this commit: robot , 11 links, 10 joints
Links:
- link foot: geometry collision capsule length=0.39000 radius=0.06000; visual capsule length=0.39000 radius=0.06000
- link leg: geometry collision capsule length=0.50000 radius=0.04000; visual capsule length=0.50000 radius=0.04000
- link thigh: geometry collision capsule length=0.45000 radius=0.05000; visual capsule length=0.45000 radius=0.05000
- link torso: geometry collision capsule length=0.40000 radius=0.05000; visual capsule length=0.40000 radius=0.05000
